Commit message: newer robot + trajectories working in ros

File: src/bartender_description/urdf/bartender_description.urdf (robot description, URDF)
Before this commit: robot bartender_description, 7 links, 6 joints
Links:
- link Axis_1_link: mass 1.82885153997862 -> 1.82910817949668
- link Axis_2_link: mass 0.759061020793129 -> 1.04847679276997
- link Axis_3_link: mass 3.93214824777397 -> 0.0558365041968776
- link Axis_4_link: mass 0.856489560610893 -> 0.843880324194983
- link Axis_5_link: mass 0.0617503556433187 -> 0.0660564110907996
- link Axis_6_link: mass 0.00888214913786918 -> 0.133229676705801
- link base_link: mass 0.676504739832433 -> 0.673093868047935
Joints:
- joint Axis_1_joint: axis 1 0 0 -> 0 0 1; origin xyz=0 0 0 rpy=0 0 0 -> xyz=0 0 0.1016 rpy=-3.1416 0 3.1416
- joint Axis_2_joint: axis 0 -1 0 -> 0 0 1; limit lower=-0.69813 upper=1.7453 effort=0 velocity=0 -> lower=-1.5707 upper=1.5707 effort=0 velocity=0; origin xyz=0.137795000103731 0 -0.0646429999999996 rpy=1.5707963267949 0 -1.04721351667053 -> xyz=0.077929 2E-05 -0.1378 rpy=0 1.5708 0
- joint Axis_3_joint: axis 0 1 0 -> 0 0 1; limit lower=-0.87267 upper=0.17453 effort=0 velocity=0 -> lower=0 upper=2.09 effort=0 velocity=0; origin xyz=0 0 -0.457236661597999 rpy=-3.14159265358979 1.02839101554935 0 -> xyz=0.45724 -1.27E-05 -0.058371 rpy=-3.1416 0 1.5708
- joint Axis_4_joint: axis 0 0 -1 -> 0 0 1; origin xyz=0.00833174747644083 -0.0641349999999993 -0.2046669392351 rpy=-3.1227709049678 -0.000168316999353158 -1.56185493455129 -> xyz=0.1630924711265 -0.0889905536771165 0.0190500000000004 rpy=-2.18798771833526 -1.57079630572147 1.65009985822568
- joint Axis_5_joint: axis 1 0 0 -> 0 0 -1; origin xyz=-0.217825000000417 0 0.17718532 rpy=0 0 0 -> xyz=-0.0173250000739991 0 -0.196235319999999 rpy=-1.5707963267949 0 1.5707963267949
- joint Axis_6_joint: origin xyz=0.2205 0 0.0283074999999999 rpy=3.14159265358979 0 -0.137857887972684 -> xyz=0 0.0170000000000001 -0.021 rpy=1.5707963267949 1.5707963267949 0
